File: PD_ElectrodeBoard_v6.sch (KiCad schematic (older format))
At the start: 125 parts, among them J1 Conn_02x32_Odd_Even, J11 TopPlate, J2 Conn_02x32_Odd_Even, X1 DMFElectrode

Commit message: Finished layout
Parts:
- removed G3: AprilTag, PurpleDrop:tag36_11_00006_6.00mm, symbol PurpleDrop:AprilTag
- added X5: DMFElectrode, PurpleDrop:SimplePad, symbol Electrodes:DMFElectrode
- G1: footprint PurpleDrop:tag36_11_00004_6.00mm -> PurpleDrop:tag36_11_00007_6.00mm
- G2: footprint PurpleDrop:tag36_11_00005_6.00mm -> PurpleDrop:tag36_11_00008_6.00mm
- J11: footprint PurpleDrop:TopPlatePad -> PurpleDrop:Header1_RA
- gave numbers to parts that had none: 3
Connections:
- net P89: now also X5.1
Changed lines of the file:
@@
 F 0 "J11" H 8680 5892 50  0000 L CNN
 F 1 "TopPlate" H 8680 5801 50  0000 L CNN
-F 2 "PurpleDrop:TopPlatePad" H 8600 5850 50  0001 C CNN
+F 2 "PurpleDrop:Header1_RA" H 8600 5850 50  0001 C CNN
 F 3 "~" H 8600 5850 50  0001 C CNN
 	1    8600 5850
@@
 F 0 "G1" H 1528 6671 50  0000 L CNN
 F 1 "AprilTag" H 1528 6580 50  0000 L CNN
-F 2 "PurpleDrop:tag36_11_00004_6.00mm" H 1350 6600 50  0001 C CNN
+F 2 "PurpleDrop:tag36_11_00007_6.00mm" H 1350 6600 50  0001 C CNN
 F 3 "" H 1350 6600 50  0001 C CNN
 	1    1350 6600
@@
 F 0 "G2" H 2228 6671 50  0000 L CNN
 F 1 "AprilTag" H 2228 6580 50  0000 L CNN
-F 2 "PurpleDrop:tag36_11_00005_6.00mm" H 2050 6600 50  0001 C CNN
+F 2 "PurpleDrop:tag36_11_00008_6.00mm" H 2050 6600 50  0001 C CNN
 F 3 "" H 2050 6600 50  0001 C CNN
 	1    2050 6600
-	1    0    0    -1
-$EndComp
-$Comp
-L PurpleDrop:AprilTag G3
-U 1 1 5F5CC3E4
-P 2750 6600
-F 0 "G3" H 2928 6671 50  0000 L CNN
-F 1 "AprilTag" H 2928 6580 50  0000 L CNN
-F 2 "PurpleDrop:tag36_11_00006_6.00mm" H 2750 6600 50  0001 C CNN
-F 3 "" H 2750 6600 50  0001 C CNN
-	1    2750 6600
 	1    0    0    -1
 $EndComp
@@
 P88
 $Comp
-L Electrodes:DMFElectrode X?
+L Electrodes:DMFElectrode X4
 U 1 1 606AA665
 P 6300 4850
-F 0 "X?" H 6428 5096 50  0000 L CNN
+F 0 "X4" H 6428 5096 50  0000 L CNN
 F 1 "DMFElectrode" H 6428 5005 50  0001 L CNN
 F 2 "PurpleDrop:SimplePad" H 6300 4850 50  0001 C CNN
@@
 $EndComp
 $Comp
-L Electrodes:DMFElectrode X?
+L Electrodes:DMFElectrode X3
 U 1 1 606AB2BC
 P 6300 4700
-F 0 "X?" H 6428 4946 50  0000 L CNN
+F 0 "X3" H 6428 4946 50  0000 L CNN
 F 1 "DMFElectrode" H 6428 4855 50  0001 L CNN
 F 2 "PurpleDrop:SimplePad" H 6300 4700 50  0001 C CNN
@@
 $EndComp
 $Comp
-L Electrodes:DMFElectrode X?
+L Electrodes:DMFElectrode X2
 U 1 1 606ABDF5
 P 6300 4550
-F 0 "X?" H 6428 4796 50  0000 L CNN
+F 0 "X2" H 6428 4796 50  0000 L CNN
 F 1 "DMFElectrode" H 6428 4705 50  0001 L CNN
 F 2 "PurpleDrop:SimplePad" H 6300 4550 50  0001 C CNN
@@
 Wire Wire Line
 	6150 4500 6150 4650
+$Comp
+L Electrodes:DMFElectrode X5
+U 1 1 60713C8C
+P 6350 5450
+F 0 "X5" H 6478 5696 50  0000 L CNN
+F 1 "DMFElectrode" H 6478 5605 50  0001 L CNN
+F 2 "PurpleDrop:SimplePad" H 6350 5450 50  0001 C CNN
+F 3 "" H 6350 5450 50  0001 C CNN
+	1    6350 5450
+	1    0    0    -1
+$EndComp
+Wire Wire Line
+	6250 5250 5900 5250
+Text Label 5900 5250 0    50   ~ 0
+P89
 $EndSCHEMATC

Commit message: Rev 6.1 update
Parts:
- G1: footprint PurpleDrop:tag36_11_00007_6.00mm -> PurpleDrop:tag36_11_00009_8.00mm
- G2: footprint PurpleDrop:tag36_11_00008_6.00mm -> PurpleDrop:tag36_11_00010_8.00mm
Changed lines of the file:
@@
 F 0 "G1" H 1528 6671 50  0000 L CNN
 F 1 "AprilTag" H 1528 6580 50  0000 L CNN
-F 2 "PurpleDrop:tag36_11_00007_6.00mm" H 1350 6600 50  0001 C CNN
+F 2 "PurpleDrop:tag36_11_00009_8.00mm" H 1350 6600 50  0001 C CNN
 F 3 "" H 1350 6600 50  0001 C CNN
 	1    1350 6600
@@
 F 0 "G2" H 2228 6671 50  0000 L CNN
 F 1 "AprilTag" H 2228 6580 50  0000 L CNN
-F 2 "PurpleDrop:tag36_11_00008_6.00mm" H 2050 6600 50  0001 C CNN
+F 2 "PurpleDrop:tag36_11_00010_8.00mm" H 2050 6600 50  0001 C CNN
 F 3 "" H 2050 6600 50  0001 C CNN
 	1    2050 6600
