File: PD_ElectrodeBoard_v6.kicad_pcb (KiCad board)
At the start: 2 copper layers, 100 x 75 mm, 125 parts, among them J1 Conn_02x32_Odd_Even, J11 TopPlate, J2 Conn_02x32_Odd_Even, X1 DMFElectrode, X2 DMFElectrode, X3 DMFElectrode, X4 DMFElectrode, X5 DMFElectrode

Commit message: Design 6.2
Parts:
- added E112: DMFElectrode, electrode_E112, F.Cu at (218.8, 72.4)
- added E113: DMFElectrode, electrode_E113, F.Cu at (218.8, 79.9)
- added E114: DMFElectrode, electrode_E114, F.Cu at (218.8, 79.9)
- added E115: DMFElectrode, electrode_E115, F.Cu at (218.8, 79.9)
- G1: footprint PurpleDrop:tag36_11_00009_8.00mm -> PurpleDrop:tag36_11_00011_8.00mm
- G2: footprint PurpleDrop:tag36_11_00010_8.00mm -> PurpleDrop:tag36_11_00012_8.00mm
- moved E100 50.4 mm to (223.1, 100.5), turned to 0 degrees
- moved E101 50.4 mm to (223.1, 100.5), turned to 0 degrees
- moved E102 50.4 mm to (223.1, 100.5), turned to 0 degrees
- moved E103 46.7 mm to (223.1, 100.5), turned to 0 degrees
- moved E107 38.2 mm to (181.2, 79.9), turned to -90 degrees
- moved E108 38.2 mm to (181.2, 79.9), turned to -90 degrees
- moved E106 37.5 mm to (181.2, 72.4), turned to -90 degrees
- moved E109 37.5 mm to (181.2, 79.9), turned to -90 degrees
- moved E82 12.5 mm to (173.1, 100.5)
- moved E86 12.5 mm to (185.6, 100.5)
- moved E87 12.5 mm to (185.6, 100.5)
- moved E90 12.5 mm to (198.1, 100.5)
- moved E91 12.5 mm to (198.1, 100.5)
- moved E92 12.5 mm to (198.1, 100.5)
- moved E94 12.5 mm to (210.6, 100.5)
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Connections:
- E1 pad 1: (no net) -> /P54
- E10 pad 1: (no net) -> /P59
- E100 pad 1: (no net) -> /P82
- E101 pad 1: (no net) -> /P83
- E102 pad 1: (no net) -> /P81
- E103 pad 1: (no net) -> /P76
- E104 pad 1: (no net) -> /P11
- E105 pad 1: (no net) -> /P13
- E106 pad 1: (no net) -> /P12
- E107 pad 1: (no net) -> /P5
- E108 pad 1: (no net) -> /P7
- E109 pad 1: (no net) -> /P6
- E11 pad 1: (no net) -> /P63
- E110 pad 1: (no net) -> /P116
- E111 pad 1: (no net) -> /P114
- E12 pad 1: (no net) -> /P124
- E13 pad 1: (no net) -> /P126
- E14 pad 1: (no net) -> /P65
- E15 pad 1: (no net) -> /P68
- E16 pad 1: (no net) -> /P69
- E17 pad 1: (no net) -> /P71
- E18 pad 1: (no net) -> /P77
- E19 pad 1: (no net) -> /P75
- E2 pad 1: (no net) -> /P53
- E20 pad 1: (no net) -> /P73
- E21 pad 1: (no net) -> /P72
- E22 pad 1: (no net) -> /P58
- E23 pad 1: (no net) -> /P0
- E24 pad 1: (no net) -> /P70
- E25 pad 1: (no net) -> /P52
- E26 pad 1: (no net) -> /P50
- E27 pad 1: (no net) -> /P60
- E28 pad 1: (no net) -> /P78
- E29 pad 1: (no net) -> /P74
- E3 pad 1: (no net) -> /P55
- E30 pad 1: (no net) -> /P15
- E31 pad 1: (no net) -> /P14
- E32 pad 1: (no net) -> /P9
- E33 pad 1: (no net) -> /P19
- E34 pad 1: (no net) -> /P17
- E35 pad 1: (no net) -> /P16
- E36 pad 1: (no net) -> /P22
- E37 pad 1: (no net) -> /P21
- E38 pad 1: (no net) -> /P20
- E39 pad 1: (no net) -> /P25
- E4 pad 1: (no net) -> /P56
- E40 pad 1: (no net) -> /P24
- E41 pad 1: (no net) -> /P23
- E42 pad 1: (no net) -> /P28
- E43 pad 1: (no net) -> /P27
- E44 pad 1: (no net) -> /P26
- E45 pad 1: (no net) -> /P102
- E46 pad 1: (no net) -> /P101
- E47 pad 1: (no net) -> /P100
- E48 pad 1: (no net) -> /P105
- E49 pad 1: (no net) -> /P104
- E5 pad 1: (no net) -> /P51
- E50 pad 1: (no net) -> /P103
- E51 pad 1: (no net) -> /P108
- E52 pad 1: (no net) -> /P107
- E53 pad 1: (no net) -> /P106
- E54 pad 1: (no net) -> /P111
- E55 pad 1: (no net) -> /P110
- E56 pad 1: (no net) -> /P109
- E57 pad 1: (no net) -> /P113
- E58 pad 1: (no net) -> /P112
- E59 pad 1: (no net) -> /P119
- E6 pad 1: (no net) -> /P47
- E60 pad 1: (no net) -> /P8
- E61 pad 1: (no net) -> /P1
- E62 pad 1: (no net) -> /P61
- E63 pad 1: (no net) -> /P10
- E64 pad 1: (no net) -> /P2
- E65 pad 1: (no net) -> /P62
- E66 pad 1: (no net) -> /P18
- E67 pad 1: (no net) -> /P4
- E68 pad 1: (no net) -> /P3
- E69 pad 1: (no net) -> /P99
- E7 pad 1: (no net) -> /P38
- E70 pad 1: (no net) -> /P117
- E71 pad 1: (no net) -> /P118
- E72 pad 1: (no net) -> /P123
- E73 pad 1: (no net) -> /P127
- E74 pad 1: (no net) -> /P66
- E75 pad 1: (no net) -> /P125
- E76 pad 1: (no net) -> /P64
- E77 pad 1: (no net) -> /P67
- E78 pad 1: (no net) -> /P41
- E79 pad 1: (no net) -> /P46
- E8 pad 1: (no net) -> /P37
- E80 pad 1: (no net) -> /P48
- E81 pad 1: (no net) -> /P49
- E82 pad 1: (no net) -> /P44
- E83 pad 1: (no net) -> /P39
- E84 pad 1: (no net) -> /P43
- E85 pad 1: (no net) -> /P45
- E86 pad 1: (no net) -> /P40
- E87 pad 1: (no net) -> /P42
- E88 pad 1: (no net) -> /P91
- E89 pad 1: (no net) -> /P34
- E9 pad 1: (no net) -> /P57
- E90 pad 1: (no net) -> /P35
- E91 pad 1: (no net) -> /P36
- E92 pad 1: (no net) -> /P33
- E93 pad 1: (no net) -> /P89
- E94 pad 1: (no net) -> /P86
- E95 pad 1: (no net) -> /P85
- E96 pad 1: (no net) -> /P84
- E97 pad 1: (no net) -> /P87
- E98 pad 1: (no net) -> /P79
- E99 pad 1: (no net) -> /P80
- X5 pad 1: /P89 -> /P90
Routing:
- net /P33: track 0.00 -> 86.6 mm, vias 0 -> 1
- net /P34: track 0.00 -> 84.1 mm, vias 0 -> 1
- net /P91: track 0.00 -> 81.1 mm, vias 0 -> 1
- net /P90: track 0.00 -> 73.6 mm, vias 0 -> 1
- net /P39: track 66.6 -> 46.3 mm
- net /P41: track 49.8 -> 32.7 mm
- net /P40: track 61.3 -> 51.9 mm
- net /P35: track 80.7 -> 84.9 mm
- net /P89: track 68.9 -> 65.8 mm
- net /P37: track 75.8 -> 74.6 mm
- net /P43: track 35.1 -> 34.3 mm
- net /P86: track 54.4 -> 53.8 mm
- added copper zone on F.Cu, net /P90
- removed copper zone on F.Cu, net /P89
Other:
- net class Default removed
- board text added: "PurpleDrop Electrode Board 6.2"
- board text removed: "PurpleDrop Electrode Board 6.1"
